File: EagleFiles/Numpad.brd (EAGLE design)
At the start: 117.8 x 116.8 mm, 67 parts, among them X1 52559-2492

Commit message: Readme added
Parts:
- removed COMM: SJ-43514_HEADPHONES_3.5MM_X4, my_parts:SJ-43514_HEADPHONES-3.5MM_X4
- removed R4, R5: 3.3K, resistor:0207/10
Connections:
- removed net N$51: COMM.4, R4.2, R5.1
- removed net N$52: COMM.3, R5.2
- removed net N$53: COMM.2, R4.1
- net GND: no longer COMM.1
Routing:
- net GND: track 79.0 -> 0.00 mm
- net N$53: track 48.5 -> 0.00 mm, vias 1 -> 0
- net N$51: track 47.5 -> 0.00 mm
- net N$52: track 43.4 -> 0.00 mm, vias 1 -> 0
Changed lines of the file:
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@@
 </autorouter>
 <elements>
-<element name="COMM" library="my_parts" package="SJ-43514_HEADPHONES-3.5MM_X4" value="SJ-43514_HEADPHONES_3.5MM_X4" x="53.34" y="128.27" smashed="yes" rot="R270"/>
-<element name="R4" library="resistor" package="0207/10" value="3.3K" x="45.72" y="123.19" smashed="yes" rot="R90">
-<attribute name="VALUE" x="46.355" y="120.9294" size="1.27" layer="27" ratio="10" rot="R90"/>
-</element>
-<element name="R5" library="resistor" package="0207/10" value="3.3K" x="41.91" y="123.19" smashed="yes" rot="R270">
-<attribute name="VALUE" x="41.275" y="125.4506" size="1.27" layer="27" ratio="10" rot="R270"/>
-</element>
 <element name="U$35" library="STM32F10x F4xx" package="STM32F405/415_LQFP64" value="STM32F405/415_LQFP64" x="7.62" y="6.35" smashed="yes"/>
 <element name="C1" library="resistor" library_urn="urn:adsk.eagle:library:348" package="C0603" package3d_urn="urn:adsk.eagle:package:23616/2" value="4.7uF" x="17.78" y="-8.89" smashed="yes">
@@
 </signal>
 <signal name="GND">
-<contactref element="COMM" pad="1"/>
-<wire x1="3.81" y1="116.84" x2="58.42" y2="116.84" width="0.4064" layer="16"/>
-<wire x1="58.42" y1="116.84" x2="58.42" y2="128.27" width="0.4064" layer="16"/>
-<wire x1="58.42" y1="128.27" x2="58.166" y2="128.27" width="0.4064" layer="16"/>
-<wire x1="58.42" y1="128.27" x2="71.12" y2="128.27" width="0.4064" layer="16"/>
 <polygon width="0.4064" layer="16">
 <vertex x="1.27" y="130.81"/>
@@
 <contactref element="C1" pad="2"/>
 <contactref element="C2" pad="2"/>
-<wire x1="17.36" y1="10.16" x2="3.81" y2="116.84" width="0" layer="19" extent="1-16"/>
 <wire x1="13.37" y1="3.1" x2="17.36" y2="10.16" width="0" layer="19" extent="1-1"/>
 <wire x1="13.55" y1="-3.81" x2="13.37" y2="3.1" width="0" layer="19" extent="1-1"/>
@@
 <wire x1="1.87" y1="3.1" x2="1.69" y2="-3.81" width="0" layer="19" extent="1-1"/>
 </signal>
-<signal name="N$51">
-<contactref element="R4" pad="2"/>
-<contactref element="R5" pad="1"/>
-<contactref element="COMM" pad="4"/>
-<wire x1="3.81" y1="125.73" x2="39.37" y2="125.73" width="0.4064" layer="16"/>
-<wire x1="39.37" y1="125.73" x2="39.37" y2="128.27" width="0.4064" layer="16"/>
-<wire x1="39.37" y1="128.27" x2="41.91" y2="128.27" width="0.4064" layer="16"/>
-<wire x1="41.91" y1="128.27" x2="45.72" y2="128.27" width="0.4064" layer="16"/>
-<wire x1="48.768" y1="128.27" x2="45.72" y2="128.27" width="0.4064" layer="16"/>
-</signal>
-<signal name="N$52">
-<contactref element="COMM" pad="3"/>
-<contactref element="R5" pad="2"/>
-<wire x1="41.91" y1="118.11" x2="41.91" y2="121.666" width="0.4064" layer="1"/>
-<wire x1="41.91" y1="121.666" x2="54.864" y2="121.666" width="0.4064" layer="1"/>
-<wire x1="54.864" y1="121.666" x2="54.864" y2="120.142" width="0.4064" layer="1"/>
-<wire x1="19.05" y1="115.57" x2="41.91" y2="115.57" width="0.4064" layer="16"/>
-<via x="41.91" y="115.57" extent="1-16" drill="0.6" shape="square"/>
-<wire x1="41.91" y1="115.57" x2="41.91" y2="118.11" width="0.4064" layer="1"/>
-</signal>
-<signal name="N$53">
-<contactref element="COMM" pad="2"/>
-<contactref element="R4" pad="1"/>
-<wire x1="45.72" y1="118.11" x2="45.72" y2="123.19" width="0.4064" layer="16"/>
-<wire x1="45.72" y1="123.19" x2="49.784" y2="123.19" width="0.4064" layer="16"/>
-<wire x1="21.59" y1="110.49" x2="49.53" y2="110.49" width="0.4064" layer="16"/>
-<wire x1="49.53" y1="110.49" x2="49.53" y2="115.57" width="0.4064" layer="16"/>
-<via x="49.53" y="115.57" extent="1-16" drill="0.6" shape="square"/>
-<wire x1="45.72" y1="118.11" x2="49.53" y2="118.11" width="0.4064" layer="1"/>
-<wire x1="49.53" y1="118.11" x2="49.53" y2="115.57" width="0.4064" layer="1"/>
-</signal>
 <signal name="LENCHA">

Commit message: Oled schematic added
Parts:
- added 25V_TANT_CAP: 4.7uF, rcl:C0805
- added C3, C5: 0.1uF, resistor:C0603
- added C4: 4.7uF, resistor:C0603
- added C6: 10uF, resistor:C0603
- added R1: 910k, resistor:R0603
Connections:
- new net BS1: X1.6
- new net BS2: X1.7
- new net CS#: X1.8
- new net D/C#: X1.10
- new net D0: X1.13
- new net D1: X1.14
- new net D2: X1.15
- new net D3: X1.16
- new net D4: X1.17
- new net D5: X1.18
- new net D6: X1.19
- new net D7: X1.20
- new net E/RD#: X1.12
- new net IREF: R1.1, X1.21
- new net N$7: X1.4
- new net R/W#: X1.11
- new net RES#: X1.9
- new net VCC: C5.2, C6.2, X1.23
- new net VCOMH: 25V_TANT_CAP.2, X1.22
- new net VDD: C3.2, C4.2, X1.5
- new net VLSS: 25V_TANT_CAP.1, C3.1, C4.1, C5.1, C6.1, R1.2, X1.2, X1.3
- net GND: now also X1.1, X1.24
Changed lines of the file:
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@@
 <attribute name="VALUE" x="8.255" y="-15.875" size="1.27" layer="27"/>
 </element>
-<element name="R_BOOT1" library="resistor" library_urn="urn:adsk.eagle:library:348" package="R0603" package3d_urn="urn:adsk.eagle:package:23555/2" value="47K" x="16.51" y="10.16" smashed="yes">
+<element name="R_BOOT1" library="resistor" library_urn="urn:adsk.eagle:library:348" package="R0603" package3d_urn="urn:adsk.eagle:package:23555/3" value="47K" x="16.51" y="10.16" smashed="yes">
 <attribute name="NAME" x="15.875" y="10.795" size="1.27" layer="25"/>
 <attribute name="VALUE" x="15.875" y="8.255" size="1.27" layer="27"/>
@@
 </element>
 <element name="U$60" library="my_parts" package="CHERRYMX-NN" value="CHERRY-MX1A-E1NW" x="10.16" y="-427.99" smashed="yes"/>
+<element name="C3" library="resistor" library_urn="urn:adsk.eagle:library:348" package="C0603" package3d_urn="urn:adsk.eagle:package:23616/2" value="0.1uF" x="2.54" y="-443.23" smashed="yes">
+<attribute name="NAME" x="1.905" y="-442.595" size="1.27" layer="25"/>
+<attribute name="VALUE" x="1.905" y="-445.135" size="1.27" layer="27"/>
+</element>
+<element name="C4" library="resistor" library_urn="urn:adsk.eagle:library:348" package="C0603" package3d_urn="urn:adsk.eagle:package:23616/2" value="4.7uF" x="2.54" y="-447.04" smashed="yes">
+<attribute name="NAME" x="1.905" y="-446.405" size="1.27" layer="25"/>
+<attribute name="VALUE" x="1.905" y="-448.945" size="1.27" layer="27"/>
+</element>
+<element name="C5" library="resistor" library_urn="urn:adsk.eagle:library:348" package="C0603" package3d_urn="urn:adsk.eagle:package:23616/2" value="0.1uF" x="2.54" y="-450.85" smashed="yes">
+<attribute name="NAME" x="1.905" y="-450.215" size="1.27" layer="25"/>
+<attribute name="VALUE" x="1.905" y="-452.755" size="1.27" layer="27"/>
+</element>
+<element name="C6" library="resistor" library_urn="urn:adsk.eagle:library:348" package="C0603" package3d_urn="urn:adsk.eagle:package:23616/2" value="10uF" x="2.54" y="-454.66" smashed="yes">
+<attribute name="NAME" x="1.905" y="-454.025" size="1.27" layer="25"/>
+<attribute name="VALUE" x="1.905" y="-456.565" size="1.27" layer="27"/>
+</element>
+<element name="R1" library="resistor" library_urn="urn:adsk.eagle:library:348" package="R0603" package3d_urn="urn:adsk.eagle:package:23555/3" value="910k" x="2.54" y="-462.28" smashed="yes">
+<attribute name="NAME" x="1.905" y="-461.645" size="1.27" layer="25"/>
+<attribute name="VALUE" x="1.905" y="-464.185" size="1.27" layer="27"/>
+</element>
+<element name="25V_TANT_CAP" library="rcl" library_urn="urn:adsk.eagle:library:334" package="C0805" package3d_urn="urn:adsk.eagle:package:23617/2" value="4.7uF" x="3.81" y="-468.63" smashed="yes">
+<attribute name="NAME" x="2.54" y="-467.36" size="1.27" layer="25"/>
+<attribute name="SPICEPREFIX" value="C" x="3.81" y="-468.63" size="1.778" layer="27" display="off"/>
+<attribute name="VALUE" x="2.54" y="-471.17" size="1.27" layer="27"/>
+</element>
 </elements>
 <signals>
@@
 <contactref element="C1" pad="2"/>
 <contactref element="C2" pad="2"/>
+<contactref element="X1" pad="24"/>
+<contactref element="X1" pad="1"/>
 <wire x1="13.37" y1="3.1" x2="17.36" y2="10.16" width="0" layer="19" extent="1-1"/>
 <wire x1="13.55" y1="-3.81" x2="13.37" y2="3.1" width="0" layer="19" extent="1-1"/>
@@
 <wire x1="3.39" y1="-13.97" x2="8.04" y2="-13.97" width="0" layer="19" extent="1-1"/>
 <wire x1="1.69" y1="-19.05" x2="3.39" y2="-13.97" width="0" layer="19" extent="1-1"/>
+<wire x1="4.41" y1="-28.07" x2="1.69" y2="-19.05" width="0" layer="19" extent="1-1"/>
 <wire x1="1.69" y1="-3.81" x2="3.39" y2="-13.97" width="0" layer="19" extent="1-1"/>
 <wire x1="1.87" y1="3.1" x2="1.69" y2="-3.81" width="0" layer="19" extent="1-1"/>
+<wire x1="15.91" y1="-25.27" x2="16.09" y2="-13.97" width="0" layer="19" extent="1-1"/>
 </signal>
 <signal name="LENCHA">
@@
 <wire x1="2.54" y1="-353.06" x2="2.54" y2="-374.65" width="0" layer="19" extent="1-1"/>
 </signal>
+<signal name="N$7">
+<contactref element="X1" pad="4"/>
+</signal>
+<signal name="CS#">
+<contactref element="X1" pad="8"/>
+</signal>
+<signal name="RES#">
+<contactref element="X1" pad="9"/>
+</signal>
+<signal name="D/C#">
+<contactref element="X1" pad="10"/>
+</signal>
+<signal name="R/W#">
+<contactref element="X1" pad="11"/>
+</signal>
+<signal name="E/RD#">
+<contactref element="X1" pad="12"/>
+</signal>
+<signal name="D0">
+<contactref element="X1" pad="13"/>
+</signal>
+<signal name="D1">
+<contactref element="X1" pad="14"/>
+</signal>
+<signal name="D2">
+<contactref element="X1" pad="15"/>
+</signal>
+<signal name="D3">
+<contactref element="X1" pad="16"/>
+</signal>
+<signal name="D4">
+<contactref element="X1" pad="17"/>
+</signal>
+<signal name="D5">
+<contactref element="X1" pad="18"/>
+</signal>
+<signal name="D6">
+<contactref element="X1" pad="19"/>
+</signal>
+<signal name="D7">
+<contactref element="X1" pad="20"/>
+</signal>
+<signal name="IREF">
+<contactref element="X1" pad="21"/>
+<contactref element="R1" pad="1"/>
+<wire x1="14.41" y1="-28.07" x2="1.69" y2="-462.28" width="0" layer="19" extent="1-1"/>
+</signal>
+<signal name="VCOMH">
+<contactref element="X1" pad="22"/>
+<contactref element="25V_TANT_CAP" pad="2"/>
+<wire x1="14.91" y1="-25.27" x2="4.76" y2="-468.63" width="0" layer="19" extent="1-1"/>
+</signal>
+<signal name="VCC">
+<contactref element="X1" pad="23"/>
+<contactref element="C6" pad="2"/>
+<contactref element="C5" pad="2"/>
+<wire x1="3.39" y1="-450.85" x2="3.39" y2="-454.66" width="0" layer="19" extent="1-1"/>
+<wire x1="15.41" y1="-28.07" x2="3.39" y2="-450.85" width="0" layer="19" extent="1-1"/>
+</signal>
+<signal name="VDD">
+<contactref element="X1" pad="5"/>
+<contactref element="C3" pad="2"/>
+<contactref element="C4" pad="2"/>
+<wire x1="3.39" y1="-443.23" x2="3.39" y2="-447.04" width="0" layer="19" extent="1-1"/>
+<wire x1="6.41" y1="-28.07" x2="3.39" y2="-443.23" width="0" layer="19" extent="1-1"/>
+</signal>
+<signal name="BS1">
+<contactref element="X1" pad="6"/>
+</signal>
+<signal name="BS2">
+<contactref element="X1" pad="7"/>
+</signal>
+<signal name="VLSS">
+<contactref element="X1" pad="3"/>
+<contactref element="C3" pad="1"/>
+<contactref element="C4" pad="1"/>
+<contactref element="X1" pad="2"/>
+<contactref element="C5" pad="1"/>
+<contactref element="C6" pad="1"/>
+<contactref element="R1" pad="2"/>
+<contactref element="25V_TANT_CAP" pad="1"/>
+<wire x1="3.39" y1="-462.28" x2="2.86" y2="-468.63" width="0" layer="19" extent="1-1"/>
+<wire x1="1.69" y1="-454.66" x2="3.39" y2="-462.28" width="0" layer="19" extent="1-1"/>
+<wire x1="1.69" y1="-450.85" x2="1.69" y2="-454.66" width="0" layer="19" extent="1-1"/>
+<wire x1="1.69" y1="-447.04" x2="1.69" y2="-450.85" width="0" layer="19" extent="1-1"/>
+<wire x1="1.69" y1="-443.23" x2="1.69" y2="-447.04" width="0" layer="19" extent="1-1"/>
+<wire x1="5.41" y1="-28.07" x2="1.69" y2="-443.23" width="0" layer="19" extent="1-1"/>
+<wire x1="4.91" y1="-25.27" x2="5.41" y2="-28.07" width="0" layer="19" extent="1-1"/>
+</signal>
+<signal name="N$1">
+</signal>
 </signals>
